Commit message: update urdf

File: source/unitree_rl_lab/unitree_rl_lab/assets/description/m3_description_new/urdf/260127-URDF-M3.urdf (robot description, URDF)
Before this commit: robot 260122-URDF-M3, 24 links, 23 joints
Links:
- link left_ankle_pitch_link: mass 0.138311 -> 0.696287404041183; geometry collision mesh filename=package://260127-URDF-M3/meshes/left_ankle_pitch_link.STL; visual mesh filename=package://260127-URDF-M3/meshes/left_ankle_pitch_link.STL
- link left_ankle_roll_link: mass 0.740175 -> 0.138310544328732; geometry collision mesh filename=package://260127-URDF-M3/meshes/left_ankle_roll_link.STL; visual mesh filename=package://260127-URDF-M3/meshes/left_ankle_roll_link.STL
- link left_elbow_pitch_link: mass 1.380488 -> 0.41900614731109; geometry collision mesh filename=package://260127-URDF-M3/meshes/left_elbow_pitch_link.STL; visual mesh filename=package://260127-URDF-M3/meshes/left_elbow_pitch_link.STL
- link left_elbow_yaw_link: mass 0.074639 -> 0.0746182543699227; geometry collision mesh filename=package://260127-URDF-M3/meshes/left_elbow_yaw_link.STL; visual mesh filename=package://260127-URDF-M3/meshes/left_elbow_yaw_link.STL
- link left_hip_pitch_link: mass 2.081211 -> 0.551922471554424; geometry collision mesh filename=package://260127-URDF-M3/meshes/left_hip_pitch_link.STL; visual mesh filename=package://260127-URDF-M3/meshes/left_hip_pitch_link.STL
- link left_hip_roll_link: mass 0.743713 -> 0.739263584026446; geometry collision mesh filename=package://260127-URDF-M3/meshes/left_hip_roll_link.STL; visual mesh filename=package://260127-URDF-M3/meshes/left_hip_roll_link.STL
- link left_hip_yaw_link: mass 3.384210 -> 0.932794510790649; geometry collision mesh filename=package://260127-URDF-M3/meshes/left_hip_yaw_link.STL; visual mesh filename=package://260127-URDF-M3/meshes/left_hip_yaw_link.STL
- link left_knee_link: mass 3.330887 -> 0.912189093527966; geometry collision mesh filename=package://260127-URDF-M3/meshes/left_knee_link.STL; visual mesh filename=package://260127-URDF-M3/meshes/left_knee_link.STL
- link left_shoulder_pitch_link: mass 1.230258 -> 0.280274562525926; geometry collision mesh filename=package://260127-URDF-M3/meshes/left_shoulder_pitch_link.STL; visual mesh filename=package://260127-URDF-M3/meshes/left_shoulder_pitch_link.STL
- link left_shoulder_roll_link: mass 1.407838 -> 0.457253808345519; geometry collision mesh filename=package://260127-URDF-M3/meshes/left_shoulder_roll_link.STL; visual mesh filename=package://260127-URDF-M3/meshes/left_shoulder_roll_link.STL
- link left_shoulder_yaw_link: mass 1.221030 -> 0.271009277454179; geometry collision mesh filename=package://260127-URDF-M3/meshes/left_shoulder_yaw_link.STL; visual mesh filename=package://260127-URDF-M3/meshes/left_shoulder_yaw_link.STL
- link pelvis_link: mass 5.294586 -> 2.04306601835033; geometry collision mesh filename=package://260127-URDF-M3/meshes/pelvis_link.STL; visual mesh filename=package://260127-URDF-M3/meshes/pelvis_link.STL
- link right_ankle_pitch_link: mass 0.138310 -> 0.696340365748186; geometry collision mesh filename=package://260127-URDF-M3/meshes/right_ankle_pitch_link.STL; visual mesh filename=package://260127-URDF-M3/meshes/right_ankle_pitch_link.STL
- link right_ankle_roll_link: mass 0.740175 -> 0.136732682491201; geometry collision mesh filename=package://260127-URDF-M3/meshes/right_ankle_roll_link.STL; visual mesh filename=package://260127-URDF-M3/meshes/right_ankle_roll_link.STL
- link right_elbow_pitch_link: mass 1.380522 -> 0.41900297547142; geometry collision mesh filename=package://260127-URDF-M3/meshes/right_elbow_pitch_link.STL; visual mesh filename=package://260127-URDF-M3/meshes/right_elbow_pitch_link.STL
- link right_elbow_yaw_link: mass 0.074639 -> 0.0746205577795183; geometry collision mesh filename=package://260127-URDF-M3/meshes/right_elbow_yaw_link.STL; visual mesh filename=package://260127-URDF-M3/meshes/right_elbow_yaw_link.STL
- link right_hip_pitch_link: mass 2.081211 -> 0.551930524773717; geometry collision mesh filename=package://260127-URDF-M3/meshes/right_hip_pitch_link.STL; visual mesh filename=package://260127-URDF-M3/meshes/right_hip_pitch_link.STL
- link right_hip_roll_link: mass 0.743941 -> 0.736015940193128; geometry collision mesh filename=package://260127-URDF-M3/meshes/right_hip_roll_link.STL; visual mesh filename=package://260127-URDF-M3/meshes/right_hip_roll_link.STL
- link right_hip_yaw_link: mass 3.380035 -> 0.932574304008033; geometry collision mesh filename=package://260127-URDF-M3/meshes/right_hip_yaw_link.STL; visual mesh filename=package://260127-URDF-M3/meshes/right_hip_yaw_link.STL
- link right_knee_link: mass 3.319576 -> 1.26004236737945; geometry collision mesh filename=package://260127-URDF-M3/meshes/right_knee_link.STL; visual mesh filename=package://260127-URDF-M3/meshes/right_knee_link.STL
- link right_shoulder_pitch_link: mass 1.230258 -> 0.28027699615297; geometry collision mesh filename=package://260127-URDF-M3/meshes/right_shoulder_pitch_link.S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; visual mesh filename=package://260127-URDF-M3/meshes/right_shoulder_pitch_link.S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
- link right_shoulder_roll_link: mass 1.407838 -> 0.448758597405378; geometry collision mesh filename=package://260127-URDF-M3/meshes/right_shoulder_roll_link.STL; visual mesh filename=package://260127-URDF-M3/meshes/right_shoulder_roll_link.STL
- link right_shoulder_yaw_link: mass 1.221030 -> 0.270981901020764; geometry collision mesh filename=package://260127-URDF-M3/meshes/right_shoulder_yaw_link.STL; visual mesh filename=package://260127-URDF-M3/meshes/right_shoulder_yaw_link.STL
- link torso_link: mass 8.719207 -> 0.932468210056261; geometry collision mesh filename=package://260127-URDF-M3/meshes/torso_link.STL; visual mesh filename=package://260127-URDF-M3/meshes/torso_link.STL
Joints:
- removed joint right_elbow_pitch_joint
- removed joint waist_yaw_joint
- added joint right_elbow__pitch_joint: type revolute, parent right_shoulder_yaw_link, child right_elbow_pitch_link, origin xyz=0.00054551 0 -0.073792 rpy=0 0 0, axis 0 1 0, limit lower=-2.09 upper=0.79 effort=0 velocity=0
- added joint torso_joint: type revolute, parent pelvis_link, child torso_link, origin xyz=0 0 0 rpy=0 0 0, axis 0 0 1, limit lower=-2.62 upper=2.62 effort=0 velocity=0
- joint left_ankle_pitch_joint: limit lower=-0.79 upper=0.52 effort=105 velocity=12.5664 -> lower=-0.79 upper=0.52 effort=0 velocity=0; origin xyz=0.007755 0 -0.307840 rpy=0 0 0 -> xyz=0 0 0 rpy=0 0 0; parent left_knee_link -> left_ankle_roll_link
- joint left_ankle_roll_joint: axis 1 0 0 -> 1 0 -0.00017977; limit lower=-0.3491 upper=0.3491 effort=105 velocity=12.5664 -> lower=-0.35 upper=0.35 effort=0 velocity=0; origin xyz=0 0 0 rpy=0 0 0 -> xyz=0.0077553 0 -0.30784 rpy=0 0 0; parent left_ankle_pitch_link -> left_knee_link
- joint left_elbow_pitch_joint: limit lower=-2.0944 upper=0.7854 effort=105 velocity=12.5664 -> lower=-0.79 upper=2.09 effort=0 velocity=0; origin xyz=0 0 -0.075581 rpy=0 0 0 -> xyz=0.00054551 0 -0.073792 rpy=0 0 0
- joint left_elbow_yaw_joint: limit lower=-2.88 upper=2.88 effort=105 velocity=12.5 -> lower=-2.88 upper=2.88 effort=0 velocity=0; origin xyz=0 0 -0.1685 rpy=0 0 0 -> xyz=0 0.001675 -0.1685 rpy=0 0 0
- joint left_hip_pitch_joint: limit lower=-2.6180 upper=2.6180 effort=195 velocity=11.1002 -> lower=-2.62 upper=2.62 effort=0 velocity=0; origin xyz=0 0.076042 -0.13702 rpy=-0.17453 0 0 -> xyz=0 0.076043 -0.13702 rpy=-0.17453 0 -1.6339E-05
- joint left_hip_roll_joint: axis 1 0 0 -> 1 1.6583E-05 0; limit lower=-0.1745 upper=1.0472 effort=195 velocity=11.1002 -> lower=-0.17 upper=1.05 effort=0 velocity=0; origin xyz=0 0.0646 0 rpy=0.17453 0 0 -> xyz=0 0.0646 0 rpy=0.17453 0 1.6592E-05
- joint left_hip_yaw_joint: axis 0 0 1 -> -0.00017977 0 1; limit lower=-2.6180 upper=2.6180 effort=105 velocity=12.5664 -> lower=-2.62 upper=2.62 effort=0 velocity=0; origin xyz=0.000117 0 -0.076443 rpy=0 0 0 -> xyz=0.0001166 0 -0.076443 rpy=0 0 0
- joint left_knee_joint: limit lower=-0.0873 upper=2.3562 effort=195 velocity=11.1002 -> lower=-0.09 upper=2.36 effort=0 velocity=0; origin xyz=0.000123 0 -0.216620 rpy=0 0 0 -> xyz=0.00012315 0 -0.21662 rpy=0 0 0
- joint left_shoulder_pitch_joint: limit lower=-3.3161 upper=2.2689 effort=105 velocity=12.5664 -> lower=-2.27 upper=3.31 effort=0 velocity=0; origin xyz=0.000495 0.0984 0.3095 rpy=0 0 0 -> xyz=0.00049469 0.0984 0.31878 rpy=0 0 0
- joint left_shoulder_roll_joint: limit lower=-0.2618 upper=3.1765 effort=105 velocity=12.5664 -> lower=-0.26 upper=3.17 effort=0 velocity=0
- joint left_shoulder_yaw_joint: limit lower=-2.8798 upper=2.8798 effort=105 velocity=12.5664 -> lower=-2.88 upper=2.88 effort=0 velocity=0; origin xyz=0 0 -0.124 rpy=0 0 0 -> xyz=-0.00054551 0 -0.124 rpy=0 0 0
- joint right_ankle_pitch_joint: limit lower=-0.52 upper=0.79 effort=105 velocity=12.5664 -> lower=-0.52 upper=0.79 effort=0 velocity=0; origin xyz=0.007755 0 -0.307840 rpy=0 0 0 -> xyz=0 0 0 rpy=0 0 0; parent right_knee_link -> right_ankle_roll_link
- joint right_ankle_roll_joint: axis 1 0 0 -> 1 0 -0.00017977; limit lower=-0.3491 upper=0.3491 effort=105 velocity=12.5664 -> lower=-0.35 upper=0.35 effort=0 velocity=0; origin xyz=0 0 0 rpy=0 0 0 -> xyz=0.0077553 0 -0.30784 rpy=0 0 0; parent right_ankle_pitch_link -> right_knee_link
- joint right_elbow_yaw_joint: limit lower=-2.88 upper=2.88 effort=105 velocity=12.5 -> lower=-2.88 upper=2.88 effort=0 velocity=0; origin xyz=0 0 -0.1685 rpy=0 0 0 -> xyz=0 -0.001675 -0.1685 rpy=0 0 0
- joint right_hip_pitch_joint: limit lower=-2.6180 upper=2.6180 effort=195 velocity=11.1002 -> lower=-2.62 upper=2.62 effort=0 velocity=0; origin xyz=0 -0.076042 -0.13702 rpy=0.17453 0 0 -> xyz=0 -0.076042 -0.13702 rpy=0.17453 0 -1.6395E-05
- joint right_hip_roll_joint: axis 1 0 0 -> 1 1.7201E-05 0; limit lower=-1.0472 upper=0.1745 effort=195 velocity=11.1002 -> lower=-1.05 upper=0.17 effort=0 velocity=0; origin xyz=0 -0.0646 0 rpy=-0.17453 0 0 -> xyz=0 -0.065674 0.00018983 rpy=-0.17453 0 1.6648E-05
- joint right_hip_yaw_joint: axis 0 0 1 -> -0.00017977 0 1; limit lower=-2.6180 upper=2.6180 effort=105 velocity=12.5664 -> lower=-2.62 upper=2.62 effort=0 velocity=0; origin xyz=0.000117 0 -0.076443 rpy=0 0 0 -> xyz=0.0001166 0.0010903 -0.076443 rpy=0 0 0
- joint right_knee_joint: limit lower=-0.0873 upper=2.3562 effort=195 velocity=11.1002 -> lower=-2.36 upper=0.09 effort=0 velocity=0; origin xyz=0.000123 0 -0.216620 rpy=0 0 0 -> xyz=0.00012315 0 -0.21662 rpy=0 0 0
- joint right_shoulder_pitch_joint: limit lower=-3.3161 upper=2.2689 effort=105 velocity=12.5664 -> lower=-3.31 upper=2.27 effort=0 velocity=0; origin xyz=0.000495 -0.0984 0.3095 rpy=0 0 0 -> xyz=0.00049469 -0.0984 0.31878 rpy=0 0 0
- joint right_shoulder_roll_joint: limit lower=-3.1765 upper=0.2618 effort=105 velocity=12.5664 -> lower=-3.17 upper=0.26 effort=0 velocity=0
- joint right_shoulder_yaw_joint: limit lower=-2.8798 upper=2.8798 effort=105 velocity=12.5664 -> lower=-2.88 upper=2.88 effort=0 velocity=0; origin xyz=0 0 -0.124 rpy=0 0 0 -> xyz=-0.00054551 0 -0.124 rpy=0 0 0

File: source/unitree_rl_lab/unitree_rl_lab/assets/description/m3_description_new/urdf/m3_23dof.urdf (robot description, URDF)
Before this commit: robot 260122-URDF-M3, 24 links, 23 joints
Links:
- link left_ankle_pitch_link: mass 0.138311 -> 0.740175
- link left_ankle_roll_link: mass 0.740175 -> 0.138311
- link right_ankle_pitch_link: mass 0.138310 -> 0.740175
- link right_ankle_roll_link: mass 0.740175 -> 0.138310
Joints:
- joint left_ankle_pitch_joint: origin xyz=0.007755 0 -0.307840 rpy=0 0 0 -> xyz=0 0 0 rpy=0 0 0; parent left_knee_link -> left_ankle_roll_link
- joint left_ankle_roll_joint: origin xyz=0 0 0 rpy=0 0 0 -> xyz=0.007755 0 -0.307840 rpy=0 0 0; parent left_ankle_pitch_link -> left_knee_link
- joint right_ankle_pitch_joint: origin xyz=0.007755 0 -0.307840 rpy=0 0 0 -> xyz=0 0 0 rpy=0 0 0; parent right_knee_link -> right_ankle_roll_link
- joint right_ankle_roll_joint: origin xyz=0 0 0 rpy=0 0 0 -> xyz=0.007755 0 -0.307840 rpy=0 0 0; parent right_ankle_pitch_link -> right_knee_link
