Commit message: update parallel urdf with non-extra link, non-parallel urdf woth pitch-joint first version

File: source/unitree_rl_lab/unitree_rl_lab/assets/description/m3_description/urdf/m3_23dof.urdf (robot description, URDF)
Before this commit: robot 260122-URDF-M3, 24 links, 23 joints
Joints:
- joint left_ankle_pitch_joint: limit lower=-0.79 upper=0.52 effort=105 velocity=12.5664 -> lower=-0.52 upper=0.79 effort=105 velocity=12.5664

Commit message: update urdf

File: source/unitree_rl_lab/unitree_rl_lab/assets/description/m3_description/urdf/m3_23dof.urdf (robot description, URDF)
Before this commit: robot 260122-URDF-M3, 24 links, 23 joints
Joints:
- joint left_ankle_pitch_joint: limit lower=-0.52 upper=0.79 effort=105 velocity=12.5664 -> lower=-0.79 upper=0.52 effort=105 velocity=12.5664
- joint right_ankle_pitch_joint: limit lower=-0.52 upper=0.79 effort=105 velocity=12.5664 -> lower=-0.79 upper=0.52 effort=105 velocity=12.5664

File: source/unitree_rl_lab/unitree_rl_lab/assets/description/m3_parallel_description/urdf/m3_23dof.urdf (robot description, URDF)
Before this commit: robot 260122-URDF-M3, 24 links, 23 joints
Joints:
- joint right_ankle_pitch_joint: limit lower=-0.52 upper=0.79 effort=105 velocity=12.5664 -> lower=-0.79 upper=0.52 effort=105 velocity=12.5664
